Commit message: run on noetic

File: src/racecar_description/urdf/racecar.urdf.xacro (robot description, xacro)
@@ -33,24 +33,24 @@
   <xacro:include filename="$(find racecar_description)/urdf/sensors/camera.xacro" />
   <!-- Degree-to-radian conversions -->
-  <xacro:property name="degrees_45" value="0.785398163"/>
-  <xacro:property name="degrees_90" value="1.57079633"/>
+  <xacro:property name="degrees_45" value="0.785398163" />
+  <xacro:property name="degrees_90" value="1.57079633" />
   <!-- chassis_length is measured along the x axis, chassis_width
        along the y axis, and chassis_height along the z axis. -->
-  <xacro:property name="chassis_length" value="0.258"/>
-  <xacro:property name="chassis_width" value="0.168"/>
-  <xacro:property name="chassis_height" value="0.01"/>
-  <xacro:property name="chassis_mass" value="2.788"/>
+  <xacro:property name="chassis_length" value="0.258" />
+  <xacro:property name="chassis_width" value="0.168" />
+  <xacro:property name="chassis_height" value="0.01" />
+  <xacro:property name="chassis_mass" value="2.788" />
   <!-- battery_dist is the distance between the inner edges of the
        batteries. battery_comp_depth is the battery compartment depth.
        battery_length is measured along the x axis, battery_width
        along the y axis, and battery_height along the z axis. -->
-  <xacro:property name="battery_x_offset" value="0.055"/>
-  <xacro:property name="battery_dist" value="0.065"/>
-  <xacro:property name="battery_comp_depth" value="0.02"/>
-  <xacro:property name="battery_comp_angle" value="0.34906585"/>
-  <xacro:property name="battery_length" value="0.16"/>
-  <xacro:property name="battery_width" value="0.047"/>
-  <xacro:property name="battery_height" value="0.024"/>
-  <xacro:property name="battery_mass" value="0.5025"/>
+  <xacro:property name="battery_x_offset" value="0.055" />
+  <xacro:property name="battery_dist" value="0.065" />
+  <xacro:property name="battery_comp_depth" value="0.02" />
+  <xacro:property name="battery_comp_angle" value="0.34906585" />
+  <xacro:property name="battery_length" value="0.16" />
+  <xacro:property name="battery_width" value="0.047" />
+  <xacro:property name="battery_height" value="0.024" />
+  <xacro:property name="battery_mass" value="0.5025" />
   <!-- hub_dia and tire_dia are the diameters of the hub and tire,
        respectively. hex_hub_depth is the distance that the hex hub is
@@ -58,24 +58,24 @@
        is a "zero offset" wheel. hex_hub_depth = tire_width / 2 -
        axle_length. -->
-  <xacro:property name="hub_dia" value="0.09652"/>
-  <xacro:property name="tire_dia" value="0.14605"/>
-  <xacro:property name="tire_width" value="0.0889"/>
-  <xacro:property name="hex_hub_depth" value="0.01445"/>
-  <xacro:property name="wheel_mass" value="0.29"/>
+  <xacro:property name="hub_dia" value="0.09652" />
+  <xacro:property name="tire_dia" value="0.14605" />
+  <xacro:property name="tire_width" value="0.0889" />
+  <xacro:property name="hex_hub_depth" value="0.01445" />
+  <xacro:property name="wheel_mass" value="0.29" />
   <!-- hex_hub_dist is the distance between left and right hex hubs when
        the shock absorbers are fully extended. axle_length is the distance
        from a U joint to the corresponding hex hub. wheel_travel is the
        vertical wheel travel. -->
-  <xacro:property name="wheelbase" value="0.335"/>
-  <xacro:property name="hex_hub_dist" value="0.365"/>
-  <xacro:property name="axle_length" value="0.03"/>
-  <xacro:property name="wheel_travel" value="0.084"/>
-  <xacro:property name="shock_z_offset" value="0.0655"/>
+  <xacro:property name="wheelbase" value="0.335" />
+  <xacro:property name="hex_hub_dist" value="0.365" />
+  <xacro:property name="axle_length" value="0.03" />
+  <xacro:property name="wheel_travel" value="0.084" />
+  <xacro:property name="shock_z_offset" value="0.0655" />
   <!-- shock_eff_limit is 2 * ((shock_stroke / 2) * shock_spring_constant) N.
        shock_stroke is 0.028575 meters. shock_spring_constant, an approximation
        of a Traxxas Ultra Shock shock absorber spring's constant, is
        437.817 N/m. -->
-  <xacro:property name="shock_eff_limit" value="12.5106"/>
-  <xacro:property name="shock_vel_limit" value="1000"/>
+  <xacro:property name="shock_eff_limit" value="12.5106" />
+  <xacro:property name="shock_vel_limit" value="1000" />
   <!-- The specifications for a Titan(R) 550 motor could not be found, so the
        stall torque of a Mabuchi Motor(R) RS-550VC-7525 motor was used instead.
@@ -90,27 +90,27 @@
        axle_vel_limit = (2 * pi) * (max_speed / (pi * tire_dia)) =
          244.8696 rad/s -->
-  <xacro:property name="axle_eff_limit" value="5.12766"/>
-  <xacro:property name="axle_vel_limit" value="244.8696"/>
+  <xacro:property name="axle_eff_limit" value="5.12766" />
+  <xacro:property name="axle_vel_limit" value="244.8696" />
   <!-- These constants are used to simulate a Traxxas 2056 servo operated at
        6 V. servo_stall_torque is measured in N m. servo_no_load_speed is
        measured in rad/s. -->
-  <xacro:property name="servo_stall_torque" value="0.5649"/>
-  <xacro:property name="servo_no_load_speed" value="4.553"/>
-  <xacro:property name="layer_mass"   value="0.0" />
-  <xacro:property name="layer_x" value="0.40"/>
-  <xacro:property name="layer_y" value="0.18"/>
-  <xacro:property name="layer_z" value="0.01"/>
-  <xacro:property name="layer_height" value="0.08"/>
+  <xacro:property name="servo_stall_torque" value="0.5649" />
+  <xacro:property name="servo_no_load_speed" value="4.553" />
+  <xacro:property name="layer_mass" value="0.0" />
+  <xacro:property name="layer_x" value="0.40" />
+  <xacro:property name="layer_y" value="0.18" />
+  <xacro:property name="layer_z" value="0.01" />
+  <xacro:property name="layer_height" value="0.08" />
   <material name="battery_mat">
-    <color rgba="0 0 1 1"/>
+    <color rgba="0 0 1 1" />
   </material>
   <material name="chassis_mat">
-    <color rgba="0.5 0.5 0.5 1"/>
+    <color rgba="0.5 0.5 0.5 1" />
   </material>
   <material name="tire_mat">
-    <color rgba="0 0 0 1"/>
+    <color rgba="0 0 0 1" />
   </material>
   <material name="yellow">
-    <color rgba="1 0.4 0 1"/>
+    <color rgba="1 0.4 0 1" />
   </material>
   <!-- Null inertial element. This is needed to make the model work with
@@ -118,6 +118,6 @@
   <xacro:macro name="null_inertial">
     <inertial>
-      <mass value="0.001"/>
-      <inertia ixx="0.001" ixy="0" ixz="0" iyy="0.001" iyz="0" izz="0.001"/>
+      <mass value="0.001" />
+      <inertia ixx="0.001" ixy="0" ixz="0" iyy="0.001" iyz="0" izz="0.001" />
     </inertial>
   </xacro:macro>
@@ -125,13 +125,13 @@
        along the y axis, and height along the z axis. -->
   <xacro:macro name="solid_cuboid_inertial"
-               params="width depth height mass *origin">
+    params="width depth height mass *origin">
     <inertial>
-      <xacro:insert_block name="origin"/>
-      <mass value="${mass}"/>
+      <xacro:insert_block name="origin" />
+      <mass value="${mass}" />
       <inertia ixx="${mass * (depth * depth + height * height) / 12}"
-               ixy="0" ixz="0"
-               iyy="${mass * (width * width + height * height) / 12}"
-               iyz="0"
-               izz="${mass * (width * width + depth * depth) / 12}"/>
+        ixy="0" ixz="0"
+        iyy="${mass * (width * width + height * height) / 12}"
+        iyz="0"
+        izz="${mass * (width * width + depth * depth) / 12}" />
     </inertial>
   </xacro:macro>
@@ -140,15 +140,15 @@
        outer_rad are the tube's inner and outer radii, respectively. -->
   <xacro:macro name="thick_walled_tube_inertial"
-               params="inner_rad outer_rad height mass">
+    params="inner_rad outer_rad height mass">
     <inertial>
-      <mass value="${mass}"/>
+      <mass value="${mass}" />
       <inertia ixx="${(1 / 12) * mass * (3 * (inner_rad * inner_rad +
                     outer_rad * outer_rad) + height * height)}"
-               ixy="0" ixz="0"
-               iyy="${(1 / 12) * mass * (3 * (inner_rad * inner_rad +
+        ixy="0" ixz="0"
+        iyy="${(1 / 12) * mass * (3 * (inner_rad * inner_rad +
                     outer_rad * outer_rad) + height * height)}"
-               iyz="0"
-               izz="${mass * (inner_rad * inner_rad +
-                    outer_rad * outer_rad) / 2}"/>
+        iyz="0"
+        izz="${mass * (inner_rad * inner_rad +
+                    outer_rad * outer_rad) / 2}" />
     </inertial>
   </xacro:macro>
@@ -156,37 +156,37 @@
   <xacro:macro name="battery" params="prefix reflect">
     <joint name="chassis_to_${prefix}_battery" type="fixed">
-      <parent link="chassis"/>
-      <child link="${prefix}_battery_offset"/>
+      <parent link="chassis" />
+      <child link="${prefix}_battery_offset" />
       <origin xyz="${battery_x_offset - battery_length / 2}
                    ${reflect * battery_dist / 2}
                    0"
-              rpy="${reflect * battery_comp_angle} 0 0"/>
+        rpy="${reflect * battery_comp_angle} 0 0" />
     </joint>
     <link name="${prefix}_battery_offset">
-      <xacro:null_inertial/>
+      <xacro:null_inertial />
     </link>
     <joint name="offset_to_${prefix}_battery" type="fixed">
-      <parent link="${prefix}_battery_offset"/>
-      <child link="${prefix}_battery"/>
+      <parent link="${prefix}_battery_offset" />
+      <child link="${prefix}_battery" />
       <origin xyz="0
                    ${reflect * battery_width / 2}
-                   ${(battery_height / 2) - battery_comp_depth}"/>
+                   ${(battery_height / 2) - battery_comp_depth}" />
     </joint>
     <link name="${prefix}_battery">
       <visual>
         <geometry>
-          <box size="${battery_length} ${battery_width} ${battery_height}"/>
-        </geometry>
-        <material name="battery_mat"/>
+          <box size="${battery_length} ${battery_width} ${battery_height}" />
+        </geometry>
+        <material name="battery_mat" />
       </visual>
       <collision>
         <geometry>
-          <box size="${battery_length} ${battery_width} ${battery_height}"/>
+          <box size="${battery_length} ${battery_width} ${battery_height}" />
         </geometry>
       </collision>
       <xacro:solid_cuboid_inertial
-         width="${battery_length}" depth="${battery_width}"
-         height="${battery_height}" mass="${battery_mass}">
-        <origin/>
+        width="${battery_length}" depth="${battery_width}"
+        height="${battery_height}" mass="${battery_mass}">
+        <origin />
       </xacro:solid_cuboid_inertial>
     </link>
@@ -197,14 +197,14 @@
   <!-- Shock absorber -->
   <xacro:macro name="shock"
-               params="lr_prefix fr_prefix lr_reflect fr_reflect child">
+    params="lr_prefix fr_prefix lr_reflect fr_reflect child">
     <joint name="${lr_prefix}_${fr_prefix}_shock" type="prismatic">
-      <parent link="chassis"/>
-      <child link="${child}"/>
+      <parent link="chassis" />
+      <child link="${child}" />
       <origin xyz="${fr_reflect * wheelbase / 2}
                    ${lr_reflect * ((hex_hub_dist / 2) - axle_length)}
-                   ${(wheel_travel / 2) - shock_z_offset}"/>
-      <axis xyz="0 0 -1"/>
+                   ${(wheel_travel / 2) - shock_z_offset}" />
+      <axis xyz="0 0 -1" />
       <limit lower="${-wheel_travel / 2}" upper="${wheel_travel / 2}"
-             effort="${shock_eff_limit}" velocity="${shock_vel_limit}"/>
+        effort="${shock_eff_limit}" velocity="${shock_vel_limit}" />
     </joint>
     <transmission name="${lr_prefix}_${fr_prefix}_shock_trans">
@@ -224,14 +224,14 @@
   <xacro:macro name="wheel" params="lr_prefix fr_prefix lr_reflect">
     <link name="${lr_prefix}_${fr_prefix}_axle_carrier">
-      <xacro:null_inertial/>
+      <xacro:null_inertial />
     </link>
     <!-- The left and right axles have the same axis so that identical
          rotation values cause the wheels to rotate in the same direction. -->
     <joint name="${lr_prefix}_${fr_prefix}_axle" type="continuous">
-      <parent link="${lr_prefix}_${fr_prefix}_axle_carrier"/>
-      <child link="${lr_prefix}_${fr_prefix}_wheel"/>
-      <origin rpy="${degrees_90} 0 0"/>
-      <axis xyz="0 0 -1"/>
-      <limit effort="${axle_eff_limit}" velocity="${axle_vel_limit}"/>
+      <parent link="${lr_prefix}_${fr_prefix}_axle_carrier" />
+      <child link="${lr_prefix}_${fr_prefix}_wheel" />
+      <origin rpy="${degrees_90} 0 0" />
+      <axis xyz="0 0 -1" />
+      <limit effort="${axle_eff_limit}" velocity="${axle_vel_limit}" />
     </joint>
     <transmission name="${lr_prefix}_${fr_prefix}_axle_trans">
@@ -252,9 +252,9 @@
                      ${lr_reflect * (axle_length - (tire_width /
                      2 - hex_hub_depth))}
-                     0"/>
-        <geometry>
-          <cylinder radius="${tire_dia / 2}" length="${tire_width}"/>
-        </geometry>
-        <material name="tire_mat"/>
+                     0" />
+        <geometry>
+          <cylinder radius="${tire_dia / 2}" length="${tire_width}" />
+        </geometry>
+        <material name="tire_mat" />
       </visual>
       <collision>
@@ -262,12 +262,12 @@
                      ${lr_reflect * (axle_length - (tire_width /
                      2 - hex_hub_depth))}
-                     0"/>
-        <geometry>
-          <cylinder radius="${tire_dia / 2}" length="${tire_width}"/>
+                     0" />
+        <geometry>
+          <cylinder radius="${tire_dia / 2}" length="${tire_width}" />
         </geometry>
       </collision>
       <xacro:thick_walled_tube_inertial
-          inner_rad="${hub_dia / 2}" outer_rad="${tire_dia / 2}"
-          height="${tire_width}" mass="${wheel_mass}"/>
+        inner_rad="${hub_dia / 2}" outer_rad="${tire_dia / 2}"
+        height="${tire_width}" mass="${wheel_mass}" />
     </link>
     <gazebo reference="${lr_prefix}_${fr_prefix}_wheel">
@@ -277,17 +277,17 @@
   <!-- Front wheel -->
   <xacro:macro name="front_wheel"
-               params="lr_prefix fr_prefix lr_reflect fr_reflect">
+    params="lr_prefix fr_prefix lr_reflect fr_reflect">
     <xacro:shock lr_prefix="${lr_prefix}" fr_prefix="${fr_prefix}"
-                 lr_reflect="${lr_reflect}" fr_reflect="${fr_reflect}"
-                 child="${lr_prefix}_steering_link"/>
+      lr_reflect="${lr_reflect}" fr_reflect="${fr_reflect}"
+      child="${lr_prefix}_steering_link" />
     <link name="${lr_prefix}_steering_link">
-      <xacro:null_inertial/>
+      <xacro:null_inertial />
     </link>
     <joint name="${lr_prefix}_steering_joint" type="revolute">
-      <parent link="${lr_prefix}_steering_link"/>
-      <child link="${lr_prefix}_${fr_prefix}_axle_carrier"/>
-      <axis xyz="0 0 1"/>
+      <parent link="${lr_prefix}_steering_link" />
+      <child link="${lr_prefix}_${fr_prefix}_axle_carrier" />
+      <axis xyz="0 0 1" />
       <limit lower="${-degrees_45}" upper="${degrees_45}"
-             effort="${servo_stall_torque}" velocity="${servo_no_load_speed}"/>
+        effort="${servo_stall_torque}" velocity="${servo_no_load_speed}" />
     </joint>
     <transmission name="${lr_prefix}_steering_trans">
@@ -304,20 +304,20 @@
     </transmission>
     <xacro:wheel lr_prefix="${lr_prefix}" fr_prefix="${fr_prefix}"
-                 lr_reflect="${lr_reflect}"/>
+      lr_reflect="${lr_reflect}" />
   </xacro:macro>
   <!-- Rear wheel -->
   <xacro:macro name="rear_wheel"
-               params="lr_prefix fr_prefix lr_reflect fr_reflect">
+    params="lr_prefix fr_prefix lr_reflect fr_reflect">
     <xacro:shock lr_prefix="${lr_prefix}" fr_prefix="${fr_prefix}"
-                 lr_reflect="${lr_reflect}" fr_reflect="${fr_reflect}"
-                 child="${lr_prefix}_${fr_prefix}_axle_carrier"/>
+      lr_reflect="${lr_reflect}" fr_reflect="${fr_reflect}"
+      child="${lr_prefix}_${fr_prefix}_axle_carrier" />
     <xacro:wheel lr_prefix="${lr_prefix}" fr_prefix="${fr_prefix}"
-                 lr_reflect="${lr_reflect}"/>
+      lr_reflect="${lr_reflect}" />
   </xacro:macro>
   <!-- chassis for sensors -->
   <xacro:macro name="layer" params="layer parent m x y z *joint_pose">
     <joint name="${layer}_joint" type="fixed">
-      <xacro:insert_block name="joint_pose"/>
-      <parent link="${parent}"/>
+      <xacro:insert_block name="joint_pose" />
+      <parent link="${parent}" />
       <child link="${layer}_link" />
     </joint>
@@ -337,7 +337,7 @@
       </collision>
       <xacro:solid_cuboid_inertial
-              width="${x}" depth="${y}"
-              height="${z}" mass="${m}">
-        <origin xyz="0 0 ${-z / 2}"/>
+        width="${x}" depth="${y}"
+        height="${z}" mass="${m}">
+        <origin xyz="0 0 ${-z / 2}" />
       </xacro:solid_cuboid_inertial>
     </link>
@@ -346,5 +346,5 @@
     </gazebo>
   </xacro:macro>
-  <link name="base_footprint"/>
+  <link name="base_footprint" />
   <!-- base_link must have geometry so that its axes can be displayed in
        rviz. -->
@@ -352,7 +352,7 @@
     <visual>
       <geometry>
-        <box size="0.01 0.01 0.01"/>
+        <box size="0.01 0.01 0.01" />
       </geometry>
-      <material name="chassis_mat"/>
+      <material name="chassis_mat" />
     </visual>
   </link>
@@ -361,27 +361,27 @@
   </gazebo>
   <joint name="base_footprint_to_base_link" type="fixed">
-    <parent link="base_footprint"/>
-    <child link="base_link"/>
+    <parent link="base_footprint" />
+    <child link="base_link" />
     <origin xyz="0 0 ${(wheel_travel/2)+shock_z_offset}" />
   </joint>
   <!-- Chassis -->
   <link name="chassis">
-    <visual>W
-      <origin xyz="0 0 ${-chassis_height / 2}"/>
+    <visual>
+      <origin xyz="0 0 ${-chassis_height / 2}" />
       <geometry>
-        <box size="${chassis_length} ${chassis_width} ${chassis_height}"/>
+        <box size="${chassis_length} ${chassis_width} ${chassis_height}" />
       </geometry>
-      <material name="chassis_mat"/>
+      <material name="chassis_mat" />
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
File: src/racecar_description/urdf/sensors/camera.xacro (robot description, xacro)
@@ -2,63 +2,63 @@
 <robot xmlns:xacro="http://www.ros.org/wiki/xacro" name="camera">
 	<link name="camera_link">
-	    <inertial>
-		<mass value="0.001" />
-		<origin xyz="0 0 0" />
-		<inertia ixx="0.001" ixy="0.0" ixz="0.0"
-		         iyy="0.001" iyz="0.0"
-		         izz="0.001" />
-	    </inertial>
-	    <visual>
-		<origin xyz=" 0 0 0 " rpy="1.57 0 1.57" />
-		<geometry>
-		    <mesh filename="package://racecar_description/meshes/S1030-0315.dae" scale="0.1 0.1 0.1" />
-		</geometry>
-	    </visual>
-	    <collision>
-		<origin xyz="0.0 0.0 0.0" rpy="0 0 0" />
-		<geometry>
-		    <box size="0.03 0.16 0.03" />
-		</geometry>
-	    </collision>
+		<inertial>
+			<mass value="0.001" />
+			<origin xyz="0 0 0" />
+			<inertia ixx="0.001" ixy="0.0" ixz="0.0"
+				iyy="0.001" iyz="0.0"
+				izz="0.001" />
+		</inertial>
+		<visual>
+			<origin xyz=" 0 0 0 " rpy="1.57 0 1.57" />
+			<geometry>
+				<mesh filename="package://racecar_description/meshes/S1030-0315.dae" scale="0.1 0.1 0.1" />
+			</geometry>
+		</visual>
+		<collision>
+			<origin xyz="0.0 0.0 0.0" rpy="0 0 0" />
+			<geometry>
+				<box size="0.03 0.16 0.03" />
+			</geometry>
+		</collision>
 	</link>
 	<gazebo reference="camera_link">
-	<material>Gazebo/Black</material>
+		<material>Gazebo/Black</material>
 	</gazebo>
 	<gazebo reference="camera_link">
 		<sensor type="camera" name="camera_node">
 			<pose>0 0 0 0 0 0</pose>
-		        <update_rate>30.0</update_rate>
-		        <camera name="head">
-		            <horizontal_fov>1.3962634</horizontal_fov>
-		            <image>
-		                <width>1280</width>
-		                <height>720</height>
-		                <format>R8G8B8</format>
-		            </image>
-		            <clip>
-		                <near>0.02</near>
-		                <far>300</far>
-		            </clip>
-		            <noise>
-		                <type>gaussian</type>
-		                <mean>0.0</mean>
-		                <stddev>0.007</stddev>
-		            </noise>
-		        </camera>
-		        <plugin name="gazebo_camera" filename="libgazebo_ros_camera.so">
-		            <alwaysOn>true</alwaysOn>
-		            <updateRate>0.0</updateRate>
-		            <cameraName>/camera</cameraName>
-		            <imageTopicName>image_raw</imageTopicName>
-		            <cameraInfoTopicName>camera_info</cameraInfoTopicName>
-		            <frameName>camera_link</frameName>
-		            <hackBaseline>0.07</hackBaseline>
-		            <distortionK1>0.0</distortionK1>
-		            <distortionK2>0.0</distortionK2>
-		            <distortionK3>0.0</distortionK3>
-		            <distortionT1>0.0</distortionT1>
-		            <distortionT2>0.0</distortionT2>
-		        </plugin>
-		    </sensor>
-	  </gazebo>
+			<update_rate>30.0</update_rate>
+			<camera name="head">
+				<horizontal_fov>1.3962634</horizontal_fov>
+				<image>
+					<width>1280</width>
+					<height>720</height>
+					<format>R8G8B8</format>
+				</image>
+				<clip>
+					<near>0.02</near>
+					<far>300</far>
+				</clip>
+				<noise>
+					<type>gaussian</type>
+					<mean>0.0</mean>
+					<stddev>0.007</stddev>
+				</noise>
+			</camera>
+			<plugin name="gazebo_camera" filename="libgazebo_ros_camera.so">
+				<alwaysOn>true</alwaysOn>
+				<updateRate>0.0</updateRate>
+				<cameraName>/camera</cameraName>
+				<imageTopicName>image_raw</imageTopicName>
+				<cameraInfoTopicName>camera_info</cameraInfoTopicName>
+				<frameName>camera_link</frameName>
+				<hackBaseline>0.07</hackBaseline>
+				<distortionK1>0.0</distortionK1>
+				<distortionK2>0.0</distortionK2>
+				<distortionK3>0.0</distortionK3>
+				<distortionT1>0.0</distortionT1>
+				<distortionT2>0.0</distortionT2>
+			</plugin>
+		</sensor>
+	</gazebo>
 </robot>

File: src/racecar_description/urdf/sensors/imu.xacro (robot description, xacro)
@@ -8,6 +8,6 @@
                 <origin xyz="0 0 0" />
                 <inertia ixx="0.001" ixy="0.0" ixz="0.0"
-                         iyy="0.001" iyz="0.0"
-                         izz="0.001" />
+                    iyy="0.001" iyz="0.0"
+                    izz="0.001" />
             </inertial>
             <visual>
@@ -16,5 +16,5 @@
                     <box size="0.04 0.04 0.03" />
                 </geometry>
-                <material name="black"/>
+                <material name="tire_mat" />
             </visual>
             <collision>
@@ -48,3 +48,4 @@
         </gazebo>
     </xacro:macro>
+    <xacro:imu prefix="imu" />
 </robot>
