Commit message: run on noetic

File: src/racecar_description/urdf/sensors/lidar.xacro (robot description, xacro)
@@ -8,18 +8,18 @@
                 <origin xyz="0 0 0" />
                 <inertia ixx="0.001" ixy="0.0" ixz="0.0"
-                         iyy="0.001" iyz="0.0"
-                         izz="0.001" />
+                    iyy="0.001" iyz="0.0"
+                    izz="0.001" />
             </inertial>
             <visual>
                 <origin xyz=" 0 0 0 " rpy="0 0 0" />
                 <geometry>
-                    <cylinder length="0.05" radius="0.05"/>
+                    <cylinder length="0.05" radius="0.05" />
                 </geometry>
-                <material name="black"/>
+                <material name="tire_mat" />
             </visual>
             <collision>
                 <origin xyz="0.0 0.0 0.0" rpy="0 0 0" />
                 <geometry>
-                    <cylinder length="0.06" radius="0.05"/>
+                    <cylinder length="0.06" radius="0.05" />
                 </geometry>
             </collision>
@@ -60,3 +60,4 @@
         </gazebo>
     </xacro:macro>
+    <xacro:lidar prefix="laser" />
 </robot>
